File: PhaseB_Prototype/PhaseB_Prototype.kicad_sch (KiCad schematic)
At the start: 38 parts, among them J1 USB_B_Mini, U1 CA56-12EWA, U2 74HC595, U3 ATmega32U4-A, Y1 16MHz

Commit message: Completed schematic for Phase B
Parts:
- added C12: 10nF, Capacitor_SMD:C_0201_0603Metric, symbol Device:C_Small
- added C13: 1uF, Capacitor_SMD:C_0201_0603Metric, symbol Device:C_Small
- added C14: 2.2uF, Capacitor_SMD:C_0201_0603Metric, symbol Device:C_Small
- added J2: AVR-ISP-6, Connector_PinSocket_2.54mm:PinSocket_2x03_P2.54mm_Vertical, symbol Connector:AVR-ISP-6
- added J3: Esp_Conn, Connector_PinSocket_2.54mm:PinSocket_2x04_P2.54mm_Vertical, symbol Connector_Generic:Conn_02x04_Odd_Even
- added R15, R16, R17: 22, Resistor_SMD:R_0603_1608Metric, symbol Device:R_Small
- added U4: USBLC6-2SC6, Package_TO_SOT_SMD:SOT-23-6, symbol Power_Protection:USBLC6-2SC6
- added U5: LP2985-3.3, Package_TO_SOT_SMD:SOT-23-5, symbol Regulator_Linear:LP2985-3.3
- R14: value 330 -> 1k
Connections:
- net +5V: now also U3.7 (VBUS), C13.1, J2.2 (VCC), U4.5 (VBUS), U5.1 (VIN), U5.3 (ON/~{OFF})
- net Button_1: now also U3.18 (PD0)
- net Button_2: now also U3.19 (PD1)
- net Buzzer: now also U3.27 (PD7)
- net DS: now also U3.29 (PB5)
- net Dig1: now also U3.32 (PC7)
- net Dig2: now also U3.26 (PD6)
- net Dig3: now also U3.12 (PB7)
- net Dig4: now also U3.30 (PB6)
- net GND: now also U3.33 (~{HWB}/PE2), C12.2, C13.2, C14.2, J2.6 (GND), J3.1 (Pin_1), U4.2 (GND), U5.2 (GND)
- net GREEN_LED: now also U3.25 (PD4)
- net RED_LED: now also U3.31 (PC6)
- net RST: now also J2.5 (~{RST})
- net SH_CP: now also U3.1 (PE6)
- net ST_CP: now also U3.28 (PB4)
- net at J1.2 (D-): now also R16.2
- net at J1.3 (D+): now also R15.2
- net MISO: now reaches U3.10 (PB2)
- net MISO: now also J2.1 (MISO)
- net MOSI: now reaches U3.11 (PB3)
- net MOSI: now also J2.4 (MOSI)
- net TX: now reaches U3.20 (PD2)
- net TX: now also J3.2 (Pin_2)
- net RX: now reaches U3.21 (PD3)
- net RX: now also J3.7 (Pin_7)
- net USB_D-: now reaches U3.3 (D-)
- net USB_D-: now also U4.6 (I/O1)
- net USB_D+: now reaches U3.4 (D+)
- net USB_D+: now also U4.4 (I/O2)
- net SCK: now reaches U3.9 (PB1)
- net SCK: now also J2.3 (SCK)
- new net: J3.5 (Pin_5), R17.1
- new net: C12.1, U5.4 (BP)
- new net +3.3V: C14.1, J3.4 (Pin_4), J3.6 (Pin_6), J3.8 (Pin_8), R17.2, U5.5 (VOUT)
- new net USB_CONN_D+: R15.1, U4.3 (I/O2)
- new net USB_CONN_D-: R16.1, U4.1 (I/O1)
- no-connect marks 6 -> 16
Other:
- note added: "ESP_CONN"
- note added: "ISP Programmer"
- note added: "Voltage Regulator"
- title: PhaseB Prototype -> Phase B Prototype
- moved on the sheet: C1, C10, C11, C2, C3, C4, C5, C6, C7, C8, C9, D1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
